File: v1.0/12keypad_v1.kicad_pcb (KiCad board)
At the start: 2 copper layers, 86.2 x 70.2 mm, 56 parts, among them J1 USB_C_Receptacle_USB2.0, SW1 KEY_1_00, SW10 KEY_10_21, SW11 KEY_11_22, SW12 KEY_12_23, SW13 SW_SPDT, SW2 KEY_2_01, SW3 KEY_3_02, SW4 KEY_4_03, SW5 KEY_5_10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

Commit message: add complete v1.0
Parts:
- C12, C13: value 10p -> 30p
- H1, H2, H3, H4: footprint MountingHole:MountingHole_2.7mm_M2.5 -> MountingHole:MountingHole_2.2mm_M2
- moved SW1 68.7 mm to (116.6, 59.7), turned to 180 degrees
- moved SW12 68.7 mm to (59.4, 97.8), turned to 180 degrees
- moved SW4 68.7 mm to (59.4, 59.7), turned to 180 degrees
- moved SW9 68.7 mm to (116.6, 97.8), turned to 180 degrees
- moved SW5 57.1 mm to (116.6, 78.7), turned to 180 degrees
- moved SW8 57.1 mm to (59.4, 78.7), turned to 180 degrees
- moved SW10 42.6 mm to (97.5, 97.8), turned to 180 degrees
- moved SW11 42.6 mm to (78.5, 97.8), turned to 180 degrees
- moved SW2 42.6 mm to (97.5, 59.7), turned to 180 degrees
- moved SW3 42.6 mm to (78.5, 59.7), turned to 180 degrees
- moved SW6 19.0 mm to (97.5, 78.7), turned to 180 degrees
- moved SW7 19.0 mm to (78.5, 78.7), turned to 180 degrees
- moved D2 13.4 mm to (95.0, 64.4), turned to 90 degrees
- moved D1 13.3 mm to (114.0, 64.4), turned to 90 degrees
- moved D4 5.88 mm to (56.9, 64.4), turned to 90 degrees
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Routing:
- net VBUS: track 37.1 -> 7.96 mm, vias 2 -> 0
- net Net-(D3-Pad2): track 17.1 -> 8.13 mm, vias 2 -> 0
- net +3V3: track 139.9 -> 147.5 mm
- net Net-(D4-Pad2): track 15.4 -> 8.13 mm
- net GND: track 136.8 -> 129.6 mm, vias 12 -> 11
- net Net-(D10-Pad2): track 13.9 -> 8.13 mm
- net Net-(D9-Pad2): track 13.9 -> 8.13 mm
- net Net-(D11-Pad2): track 13.9 -> 8.13 mm
- net Net-(D12-Pad2): track 13.8 -> 8.13 mm
- net Net-(D7-Pad2): track 13.6 -> 8.13 mm
- net Net-(D6-Pad2): track 13.6 -> 8.13 mm
- net Net-(D8-Pad2): track 13.6 -> 8.13 mm
- net Net-(D5-Pad2): track 13.6 -> 8.13 mm
- net /QSPI_SD2: track 43.6 -> 38.7 mm
- net Net-(D1-Pad2): track 3.40 -> 8.13 mm
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Other:
- board text added: "Designed by: Tommaso Gualtierotti Matteo Zodi v1.0"
- board text removed: "Designed by: Tommaso Gualtierotti Matteo Zodi"
